File: 4ch_RF_FE_KiCad/RF_channel.sch (KiCad schematic (older format))
At the start: 8 parts

Commit message: initial completion of schematic capture
Parts:
- removed C?: 470pF, Capacitor_SMD:C_0402_1005Metric, symbol Device:C
- removed D?: PGB1010402KR, Diode_SMD:D_0402_1005Metric, symbol jcg_custom_parts:PGB1010402KR
- removed U?: ADL5611ARKZ-R7, RK_3, symbol ADL5611ARKZ-R7:ADL5611ARKZ-R7
- removed U?: PHA-1+, symbol jcg_custom_parts:PHA-1+
- removed U? (x3): BGS12SN6, jcg_custom:BGS12SN6, symbol jcg_custom_parts:BGS12SN6
- added C34, C35, C36, C40, C41, C47, C48, C49, C50, C51, C52, C53, C54, C56, C57, C58: 330pF, Capacitor_SMD:C_0402_1005Metric, symbol Device:C
- added C37, C43: 68pF, Capacitor_SMD:C_0402_1005Metric, symbol Device:C
- added C38, C44, C55, C59: 0.1µF, Capacitor_SMD:C_0402_1005Metric, symbol Device:C
- added C39, C45: 1.2nF, Capacitor_SMD:C_0603_1608Metric_Pad1.05x0.95mm_HandSolder, symbol Device:C
- added C42, C46: 1µF, Capacitor_SMD:C_0603_1608Metric_Pad1.05x0.95mm_HandSolder, symbol Device:C
- added F2, F3: LPF04023600L, jcg_custom:F_0402_1005Metric_2x2_LGA, symbol jcg_custom_parts:LPF04023600L
- added F4: LP0603A2140ANTR, jcg_custom:F_0603_2x2_LGA, symbol jcg_custom_parts:LP0603A2140ANTR
- added F5: DEA162300HT-8047A1, jcg_custom:F_DEA16_LGA, symbol jcg_custom_parts:DEA162300HT-8047A1
- added J4, J5, J6, J7: 5-1814832-1, digikey-footprints:RF_SMA_Vertical_5-1814832-1, symbol dk_Coaxial-Connectors-RF:5-1814832-1
- added L3, L4: 43nH, Inductor_SMD:L_0603_1608Metric_Pad1.05x0.95mm_HandSolder, symbol Device:L
- added R29: 10k, Resistor_SMD:R_0402_1005Metric, symbol Device:R_US
- added T1, T2: MABA-011082, jcg_custom:T_6pin_23_balun, symbol jcg_custom_parts:MABA-011082
- added U11, U14: ADL5611ARKZ-R7, footprints:ADL5611ARKZ-R7, symbol ADL5611ARKZ-R7:ADL5611ARKZ-R7
- added U12, U15: PE43711, Package_DFN_QFN:QFN-24-1EP_4x4mm_P0.5mm_EP2.7x2.7mm, symbol jcg_custom_parts:PE43711
- added U13, U16, U17: HMC544AETR, Package_TO_SOT_SMD:SOT-23-6_Handsoldering, symbol jcg_custom_parts:HMC544AETR
- added U18: PCAL6416APW, digikey-footprints:TSSOP-24_W4.40mm, symbol jcg_custom_parts:PCAL6416APW
- gave numbers to parts that had none: 1
Connections:
- net +3V3: now also C38.1, C44.1, C55.1, C59.1, R29.1, U12.2 (Vdd), U15.2 (Vdd), U18.2 (VDD_I2C), U18.24 (VDD_P)
- net GND: now also C37.2, C38.2, C39.2, C42.2, C43.2, C44.2, C45.2, C46.2, C55.2, C59.2, F2.2 (GND), F2.4 (GND), F3.2 (GND), F3.4 (GND), F4.2 (GND), F4.4 (GND), F5.2 (GND), F5.4 (GND), J4.1, J5.1, J6.1, J7.1, T1.2, T1.3, T1.4, T2.2, T2.3, T2.4, U11.2 (GND), U12.10 (GND), U12.11 (GND), U12.12 (GND), U12.13 (GND), U12.15 (GND), U12.17 (CLK), U12.18 (SI), U12.3 (~P~/S), U12.4 (GND), U12.6 (GND), U12.7 (GND), U12.8 (GND), U12.9 (GND), U13.2 (GND), U14.2 (GND), U15.10 (GND), U15.11 (GND), U15.12 (GND), U15.13 (GND), U15.15 (GND), U15.17 (CLK), U15.18 (SI), U15.3 (~P~/S), U15.4 (GND), U15.6 (GND), U15.7 (GND), U15.8 (GND), U15.9 (GND), U16.2 (GND), U17.2 (GND), U18.12 (VSS), U18.21 (ADDR)
- net at J3.2: now also C36.2
- new net: C34.1, U11.1 (RFIN)
- new net: C40.2, L3.2, U11.3 (RFOUT)
- new net: C40.1, U15.5 (RF1)
- new net: C48.1, U16.5 (RFC)
- new net: C48.2, U15.14 (RF2)
- new net: C49.1, F4.1 (RF_IN)
- new net: C49.2, U16.3 (RF1)
- new net: C50.1, F3.1 (RF_IN)
- new net: C50.2, U16.1 (RF2)
- new net: C53.1, U17.3 (RF1)
- new net: C53.2, F4.3 (RF_OUT)
- new net: C54.1, U17.1 (RF2)
- new net: C54.2, F5.3 (RF_OUT)
- new net: C56.2, U17.5 (RFC)
- new net: C57.1, J6.2
- new net: C57.2, T2.6
- new net: C58.1, J7.2
- new net: C58.2, T2.5
- new net: C51.1, J4.2
- new net: C47.2, U14.1 (RFIN)
- new net: C41.1, L4.2, U14.3 (RFOUT)
- new net: C36.1, U13.5 (RFC)
- new net: C35.1, U12.14 (RF2)
- new net: C41.2, U12.5 (RF1)
- new net: C47.1, F2.3 (RF_OUT)
- new net: C51.2, T1.6
- new net: C52.1, J5.2
- new net: C52.2, T1.5
- new net: F3.3 (RF_OUT), F5.1 (RF_IN)
- new net: F2.1 (RF_IN), T1.1
- new net: R29.2, U18.3 (~RESET)
- new net +5V_REG: C37.1, C39.1, C42.1, C43.1, C45.1, C46.1, L3.1, L4.1
- new net C0.25_RX: U15.1 (C0.25), U18.5 (P0_1)
- new net C0.25_TX: U12.1 (C0.25), U18.14 (P1_1)
- new net C0.5_RX: U15.24 (C0.5), U18.6 (P0_2)
- new net C0.5_TX: U12.24 (C0.5), U18.15 (P1_2)
- new net C16_RX: U15.19 (C16), U18.11 (P0_7)
- new net C16_TX: U12.19 (C16), U18.20 (P1_7)
- new net C1_RX: U15.23 (C1), U18.7 (P0_3)
- new net C1_TX: U12.23 (C1), U18.16 (P1_3)
- new net C2_RX: U15.22 (C2), U18.8 (P0_4)
- new net C2_TX: U12.22 (C2), U18.17 (P1_4)
- new net C4_RX: U15.21 (C4), U18.9 (P0_5)
- new net C4_TX: U12.21 (C4), U18.18 (P1_5)
- new net C8_RX: U15.20 (C8), U18.10 (P0_6)
- new net C8_TX: U12.20 (C8), U18.19 (P1_6)
- new net I2C_SCL_ATTN: U18.22 (SCL)
- new net I2C_SDA_ATTN: U18.23 (SDA)
- new net LE_RX: U15.16 (LE), U18.4 (P0_0)
- new net LE_TX: U12.16 (LE), U18.13 (P1_0)
- new net RX_FILTER_OUT: C56.1, T2.1
- new net RX_IN: C34.2, U13.3 (RF1)
- new net TX_OUT: C35.2, U13.1 (RF2)
- new net ~1ST_NYQ~_2ND_NYQ_SW: U16.6 (A), U17.6 (A)
- new net ~1ST_NYQ~_2ND_NYQ_SW_INV: U16.4 (B), U17.4 (B)
- new net ~RX~_TX_SW: U13.6 (A)
- new net ~RX~_TX_SW_INV: U13.4 (B)
- no-connect marks 0 -> 1
Other:
- note added: "1st Nyquist Zone Filter\n LPF Passband (-1dB): 0 - 2.14 GHz"
- note added: "2nd Nyquist Zone Filter\nComposite Bandpass Filter: 2.3 - 3.6 GHz\n LPF Passband (-1dB): 0 - 3.6 GHz\n HPF Passband (-1dB): > 2.3 GHz"
- note added: "7-bit (0.25dB) DSA\nAttn: 0 - 31.75 dB\nBW: 9 kHz - 6 GHz"
- note added: "ADDR: 0x20"
- note added: "DC Bias Max Power Draw: 124 mA"
- note added: "Gain: 22.2 dB\nBW: 30 - 6000 MHz\nP1dB: 21.0 dBm @ 900 MHz\nOIP3: 40.0 dBm @ 900 MHz"
- note added: "I2C GPIO Expander"
- note added: "LPF Passband (-1dB): 0 - 3.6 GHz"
- note added: "RFC-RF1: A=0,B=1\nRFC-RF2: A=1,B=0\nP1dB = 39 dBm\nt_switch = 30 ns"
- note added: "RX Differential Output"
- note added: "RX Path"
- note added: "RX/TX SMA"
- note added: "TX Differential Input"
- note added: "TX Path"
- moved on the sheet: J3

Commit message: RF layout
Signed-off-by: Gentile, John <johncgentile17@gmail.com>
Connections:
- net ~1ST_NYQ~_2ND_NYQ_SW: now also U16.4 (B); no longer U16.6 (A)
- net ~1ST_NYQ~_2ND_NYQ_SW_INV: now also U16.6 (A); no longer U16.4 (B)
- net at C49.2: now also U16.1 (RF2); no longer U16.3 (RF1)
- net at C50.2: now also U16.3 (RF1); no longer U16.1 (RF2)
Changed lines of the file:
@@
 	9200 2950 8900 2950
-Wire Wire Line
-	8900 3050 9000 3050
-Wire Wire Line
-	9000 3050 9000 3300
-Wire Wire Line
-	9000 3300 9450 3300
 Wire Wire Line
 	10800 3050 10900 3050
@@
 Wire Wire Line
 	11350 3450 11600 3450
-Wire Wire Line
-	8900 2850 9300 2850
-Wire Wire Line
-	9300 2850 9300 2500
-Wire Wire Line
-	9300 2500 9450 2500
 $Comp
 L power:GND #PWR070
@@
 Text Notes 13450 6350 0    118  ~ 24
 I2C GPIO Expander
-Text HLabel 7700 3250 0    50   Input Italic 0
-~1ST_NYQ~_2ND_NYQ_SW
 Text Notes 8100 3450 0    50   Italic 0
 RFC-RF1: A=0,B=1\nRFC-RF2: A=1,B=0\nP1dB  = 39 dBm\nt_switch  = 30 ns
@@
 	1    0    0    -1
 $EndComp
-Text Notes 5600 3550 0    50   Italic 0
+Text Notes 5450 3550 0    50   Italic 0
 7-bit (0.25dB) DSA\nAttn: 0 - 31.75 dB\nBW: 9 kHz - 6 GHz
 Text Notes 2500 9000 0    50   Italic 0
 7-bit (0.25dB) DSA\nAttn: 0 - 31.75 dB\nBW: 9 kHz - 6 GHz
-Text HLabel 8000 2300 2    50   Input Italic 0
-~1ST_NYQ~_2ND_NYQ_SW_INV
 Wire Wire Line
 	8000 2850 7750 2850
@@
 F 3 "http://www.psemi.com/pdf/datasheets/pe43711ds.pdf" H 5900 2600 50  0001 C CNN
 F 4 "1046-1138-1-ND" H 6300 3450 50  0001 C CNN "Digi-Key PN"
-F 5 "RF ATTENUATOR 31.5DB 50OHM 24QFN" H 5200 1750 50  0000 L CNN "Description"
+F 5 "RF ATTENUATOR 31.5DB 50OHM 24QFN" H 4750 1750 50  0000 L CNN "Description"
 	1    6300 2500
 	1    0    0    -1
@@
 	-1   0    0    -1
 $EndComp
+Text HLabel 7700 3250 0    50   Input Italic 0
+~1ST_NYQ~_2ND_NYQ_SW_INV
+Text HLabel 8000 2300 2    50   Input Italic 0
+~1ST_NYQ~_2ND_NYQ_SW
+Wire Wire Line
+	9450 3300 9350 3300
+Wire Wire Line
+	9350 3300 9350 2850
+Wire Wire Line
+	9350 2850 8900 2850
+Wire Wire Line
+	9450 2500 9100 2500
+Wire Wire Line
+	9100 2500 9100 3050
+Wire Wire Line
+	8900 3050 9100 3050
 $EndSCHEMATC
