File: 4ch_RF_FE_KiCad/4ch_RF_FE_KiCad.kicad_pcb (KiCad board)
At the start: 2 copper layers, 272 parts, among them J1 PJ1-021-SMT-TR, J10 5-1814832-1, J11 5-1814832-1, J12 5-1814832-1, J13 5-1814832-1, J14 5-1814832-1, J15 5-1814832-1, J16 5-1814832-1, J17 5-1814832-1, J18 5-1814832-1, J19 5-1814832-1, J2 PPTC062LJBN-RC, J20 5-1814832-1, J21 5-1814832-1, J22 5-1814832-1, J3 5-1814832-1, J4 5-1814832-1, J5 5-1814832-1, J6 5-1814832-1, J7 5-1814832-1, J8 5-1814832-1, J9 5-1814832-1, T1 MABA-011082, T2 MABA-011082, T3 MABA-011082, T4 MABA-011082, T5 MABA-011082, T6 MABA-011082, T7 MABA-011082, T8 MABA-011082, U1 MCP1755ST-5002E_DB, U10 SN74HCU04PWR, U11 ADL5611ARKZ-R7, U12 PE43711, U13 HMC544AETR, U14 ADL5611ARKZ-R7, U15 PE43711, U16 HMC544AETR, U17 HMC544AETR, U18 PCAL6416APW, U19 ADL5611ARKZ-R7, U2 MCP1755ST-5002E_DB, U20 PE43711, U21 HMC544AETR, U22 ADL5611ARKZ-R7, U23 PE43711, U24 HMC544AETR, U25 HMC544AETR, U26 PCAL6416APW, U27 ADL5611ARKZ-R7, U28 PE43711, U29 HMC544AETR, U3 MCP1755ST-5002E_DB, U30 ADL5611ARKZ-R7, U31 PE43711, U32 HMC544AETR, U33 HMC544AETR, U34 PCAL6416APW, U35 ADL5611ARKZ-R7, U36 PE43711, U37 HMC544AETR, U38 ADL5611ARKZ-R7, U39 PE43711, U4 MCP1755ST-5002E_DB, U40 HMC544AETR, U41 HMC544AETR, U42 PCAL6416APW, U5 INA219AIDCNR, U6 TPS562208DDCT, U7 PCA9548APW, U8 M24C02-FDW, U9 SN74LVC125APWR

Commit message: (+) starting layout
Signed-off-by: Gentile, John <johncgentile17@gmail.com>
Parts:
- added FID1: Fiducial, Fiducial:Fiducial_1mm_Mask2mm, F.Cu at (384.9, 190.1)
- added FID2: Fiducial, Fiducial:Fiducial_1mm_Mask2mm, F.Cu at (388.5, 190.1)
- added FID3: Fiducial, Fiducial:Fiducial_1mm_Mask2mm, F.Cu at (392.0, 190.1)
- added H1: MountingHole_Pad, MountingHole:MountingHole_3.7mm_Pad_Via, F.Cu at (369.7, 192.8)
- added H2: MountingHole_Pad, MountingHole:MountingHole_3.7mm_Pad_Via, F.Cu at (369.7, 201.8)
- added H3: MountingHole_Pad, MountingHole:MountingHole_3.7mm_Pad_Via, F.Cu at (378.7, 192.8)
- added H4: MountingHole_Pad, MountingHole:MountingHole_3.7mm_Pad_Via, F.Cu at (378.7, 201.8)
- J2: footprint digikey-footprints:PinHeader_2x6_P2.54mm_Vertical_SMD -> Connector_PinHeader_2.54mm:PinHeader_2x06_P2.54mm_Horizontal
- RN5: moved to B.Cu
- moved C28 157.8 mm to (227.7, 227.3)
- moved C33 157.8 mm to (233.8, 224.1)
- moved R24 157.8 mm to (240.2, 220.1)
- moved R25 157.8 mm to (236.7, 224.1)
- moved RN1 157.8 mm to (227.7, 219.0)
- moved RN3 157.8 mm to (230.8, 219.0)
- moved C31 157.8 mm to (227.3, 229.3)
- moved C32 157.8 mm to (233.5, 226.1)
- moved R10 157.8 mm to (227.7, 225.3)
- moved R16 157.8 mm to (240.2, 218.1)
- moved R17 157.8 mm to (224.4, 227.9)
- moved R18 157.8 mm to (224.4, 229.9)
- moved R19 157.8 mm to (230.2, 229.3)
- moved R20 157.8 mm to (236.4, 226.1)
- moved R21 157.8 mm to (243.1, 218.1)
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Connections:
- L1 pad 1: Net-(C3-Pad1) -> Net-(C1-Pad1)
- L1 pad 2: Net-(C1-Pad1) -> Net-(C3-Pad1)
- R5 pad 2: /Power Input & Regulation/sense12V_N -> /Power Input & Regulation/sense12V_P
- R5 pad 4: /Power Input & Regulation/sense12V_P -> /Power Input & Regulation/sense12V_N
Routing:
- net Net-(C1-Pad1): track 0.00 -> 17.5 mm
- net Net-(C3-Pad1): track 0.00 -> 8.13 mm
- net Net-(F1-Pad1): track 0.00 -> 4.36 mm
Other:
- copper layers 2 -> 4
- net class 12V_PWR added: clearance 0.127, trace_width 0.3048, via_dia 0.508, via_drill 0.254
- net class Default: clearance 0.2 -> 0.127; trace_width 0.25 -> 0.127; via_dia 0.8 -> 0.4572; via_drill 0.4 -> 0.254
- rule pad_to_mask_clearance: 0.051 -> 0.0508
- rule solder_mask_min_width: 0.25 -> 0.1016
- rule trace_clearance: 0.2 -> 0.127
- rule trace_min: 0.2 -> 0.127
- rule via_min_drill: 0.3 -> 0.254
- rule via_min_size: 0.4 -> 0.4572

Commit message: (+) power & DIO layout & impedance calcs
Signed-off-by: Gentile, John <johncgentile17@gmail.com>
Parts:
- added R30: 10k, Resistor_SMD:R_0402_1005Metric, B.Cu at (48.4, 159.6)
- C10, C12, C15, C16, C19, C20, C23, C24, C32, C6, C9, R11, R12, R13, R14, R15, R2, R21, R3, R9, U3, U4, U5, U7, U9: moved to B.Cu
- moved H1 333.4 mm to (36.7, 209.4)
- moved C29 223.7 mm to (40.0, 183.8)
- moved J2 223.0 mm to (43.8, 201.0), turned to 180 degrees
- moved FB1 218.6 mm to (42.5, 184.5), turned to 0 degrees
- moved C30 215.6 mm to (42.2, 180.7), turned to 180 degrees
- moved R15 215.5 mm to (47.5, 203.8), turned to 270 degrees
- moved R11 215.5 mm to (47.4, 193.0), turned to 90 degrees
- moved R12 215.2 mm to (47.5, 198.1)
- moved R9 214.8 mm to (47.9, 195.2), turned to 180 degrees
- moved R14 214.8 mm to (48.0, 201.9), turned to 180 degrees
- moved R13 214.6 mm to (48.0, 200.3), turned to 0 degrees
- moved RN5 206.9 mm to (52.1, 198.4), turned to 0 degrees
- moved RN4 206.5 mm to (51.9, 198.4), turned to 180 degrees
- moved R20 194.3 mm to (46.6, 184.5), turned to 90 degrees
- moved R24 191.5 mm to (52.2, 183.5), turned to 270 degrees
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Connections:
- net Net-(C11-Pad1) renamed /Power Input & Regulation/PWR_IN_CMC
- net Net-(C26-Pad2) renamed /Power Input & Regulation/V_SW_NODE
- net Net-(F1-Pad1) renamed /Power Input & Regulation/PWR_IN
- net Net-(R16-Pad1) renamed /Digitial I/O via PMOD/~RX~_TX_SW1_BUF
- net Net-(R17-Pad1) renamed /Digitial I/O via PMOD/~RX~_TX_SW1_INV_BUF
- net Net-(R18-Pad1) renamed /Digitial I/O via PMOD/~RX~_TX_SW0_BUF
- net Net-(R19-Pad1) renamed /Digitial I/O via PMOD/~RX~_TX_SW0_INV_BUF
- net Net-(R20-Pad1) renamed /Digitial I/O via PMOD/~RX~_TX_SW2_INV_BUF
- net Net-(R21-Pad2) renamed /Digitial I/O via PMOD/~RX~_TX_SW3_INV_BUF
- net Net-(R22-Pad2) renamed /Digitial I/O via PMOD/~RX~_TX_SW3_BUF
- net Net-(R24-Pad2) renamed /Digitial I/O via PMOD/~RX~_TX_SW2_BUF
- net Net-(R7-Pad2) renamed /Power Input & Regulation/V_FB
- C1 pad 1: Net-(C1-Pad1) -> /Power Input & Regulation/PWR_RETURN
- C2 pad 2: Net-(C1-Pad1) -> /Power Input & Regulation/PWR_RETURN
- C3 pad 1: Net-(C3-Pad1) -> /Power Input & Regulation/PWR_IN_FUSED
- C3 pad 2: Net-(C1-Pad1) -> /Power Input & Regulation/PWR_RETURN
- C4 pad 1: Net-(C1-Pad1) -> /Power Input & Regulation/PWR_RETURN
- C4 pad 2: Net-(C3-Pad1) -> /Power Input & Regulation/PWR_IN_FUSED
- F1 pad 2: Net-(C3-Pad1) -> /Power Input & Regulation/PWR_IN_FUSED
- J1 pad 2: Net-(C1-Pad1) -> /Power Input & Regulation/PWR_RETURN
- J1 pad 3: Net-(C1-Pad1) -> /Power Input & Regulation/PWR_RETURN
- L1 pad 1: Net-(C1-Pad1) -> /Power Input & Regulation/PWR_IN_FUSED
- L1 pad 2: Net-(C3-Pad1) -> /Power Input & Regulation/PWR_RETURN
- R1 pad 2: Net-(C1-Pad1) -> /Power Input & Regulation/PWR_RETURN
- U6 pad 5: /Power Input & Regulation/Vin_unreg -> Net-(R30-Pad1)
Routing:
- net /Digitial I/O via PMOD/~RX~_TX_SW3_PMOD: track 0.00 -> 53.0 mm, vias 0 -> 1
- net /Digitial I/O via PMOD/~RX~_TX_SW2_PMOD: track 0.00 -> 46.2 mm, vias 0 -> 2
- net /Digitial I/O via PMOD/~RX~_TX_SW0_PMOD: track 0.00 -> 34.8 mm, vias 0 -> 2
- net /Digitial I/O via PMOD/~RX~_TX_SW1_PMOD: track 0.00 -> 27.6 mm, vias 0 -> 2
- net GND: track 0.00 -> 24.8 mm, vias 0 -> 27
- net /Digitial I/O via PMOD/~1ST~_2ND_NYQ_BAND_SEL: track 0.00 -> 23.3 mm, vias 0 -> 1
- net Net-(C1-Pad1): track 17.5 -> 0.00 mm
- net +3V3: track 0.00 -> 13.0 mm, vias 0 -> 5
- net /Digitial I/O via PMOD/~RX~_TX_SW2_INV_BUF: track 0.00 -> 10.1 mm
- net Net-(R23-Pad2): track 0.00 -> 9.60 mm
- net /Power Input & Regulation/V_SW_NODE: track 0.00 -> 9.46 mm, vias 0 -> 6
- net Net-(C3-Pad1): track 8.13 -> 0.00 mm
- net /Digitial I/O via PMOD/~RX~_TX_SW1_BUF: track 0.00 -> 7.58 mm, vias 0 -> 1
- net Net-(R30-Pad1): track 0.00 -> 7.30 mm, vias 0 -> 1
- net /Power Input & Regulation/V_FB: track 0.00 -> 5.84 mm
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- added copper zone on B.Cu, net +3V3
- added copper zone on F.Cu, net /Digitial I/O via PMOD/3V3_IN
- added copper zone on F.Cu, net /Power Input & Regulation/5V5_SW
- added copper zone on F.Cu, net /Power Input & Regulation/PWR_IN
- added copper zone on F.Cu, net /Power Input & Regulation/PWR_IN_CMC
- added copper zone on F.Cu, net /Power Input & Regulation/PWR_IN_FUSED
- added copper zone on F.Cu, net /Power Input & Regulation/PWR_RETURN
- added copper zone on GND.Cu, net /Power Input & Regulation/PWR_RETURN
- added copper zone on B.Cu, net /Power Input & Regulation/V_SW_NODE
- added copper zone on F.Cu, net /Power Input & Regulation/V_SW_NODE
- added copper zone on F.Cu, net /Power Input & Regulation/Vin_unreg
- added copper zone on F.Cu, net GND
Other:
- net class 50Ohm_CPWG added: clearance 0.1524, trace_width 0.3175, via_dia 0.5207, via_drill 0.3175
- net class 50Ohm_SE_microstrip added: clearance 0.127, trace_width 0.35052, via_dia 0.55372, via_drill 0.35052
- net class 50Ohm_SE_stripline added: clearance 0.127, trace_width 0.30734, via_dia 0.51054, via_drill 0.30734

Commit message: RF layout
Signed-off-by: Gentile, John <johncgentile17@gmail.com>
Parts:
- C107, C111, C133, C137, C31, C55, C59, C81, C85, R26, R27, R28, R29, U18, U26, U34, U42, U8: moved to B.Cu
- U7: moved to F.Cu
- moved H2 351.0 mm to (39.4, 99.3)
- moved F2 158.5 mm to (93.2, 164.3), turned to 90 degrees
- moved C47 157.3 mm to (93.4, 157.0), turned to 90 degrees
- moved C52 153.8 mm to (84.8, 179.5), turned to 45 degrees
- moved L4 153.3 mm to (97.2, 146.6), turned to 180 degrees
- moved C38 152.0 mm to (95.2, 140.1), turned to 180 degrees
- moved U14 149.0 mm to (89.6, 150.2), turned to 90 degrees
- moved C51 147.2 mm to (100.6, 179.5), turned to 135 degrees
- moved J5 145.2 mm to (82.3, 187.1), turned to 270 degrees
- moved C45 143.3 mm to (100.5, 149.6), turned to 270 degrees
- moved C35 141.7 mm to (107.9, 123.9), turned to 45 degrees
- moved F6 141.5 mm to (176.6, 164.4), turned to 90 degrees
- moved C41 141.2 mm to (94.5, 144.0), turned to 45 degrees
- moved C43 140.9 mm to (98.4, 149.4), turned to 270 degrees
- moved U12 140.1 mm to (98.2, 136.3), turned to 90 degrees
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Connections:
- C115 pad 1: /Power Input & Regulation/+5V_CH1 -> /Power Input & Regulation/+5V_CH2
- C117 pad 1: /Power Input & Regulation/+5V_CH1 -> /Power Input & Regulation/+5V_CH2
- C120 pad 1: /Power Input & Regulation/+5V_CH1 -> /Power Input & Regulation/+5V_CH2
- C121 pad 1: /Power Input & Regulation/+5V_CH1 -> /Power Input & Regulation/+5V_CH2
- C123 pad 1: /Power Input & Regulation/+5V_CH1 -> /Power Input & Regulation/+5V_CH2
- C124 pad 1: /Power Input & Regulation/+5V_CH1 -> /Power Input & Regulation/+5V_CH2
- C37 pad 1: /Power Input & Regulation/+5V_CH3 -> /Power Input & Regulation/+5V_CH0
- C39 pad 1: /Power Input & Regulation/+5V_CH3 -> /Power Input & Regulation/+5V_CH0
- C42 pad 1: /Power Input & Regulation/+5V_CH3 -> /Power Input & Regulation/+5V_CH0
- C43 pad 1: /Power Input & Regulation/+5V_CH3 -> /Power Input & Regulation/+5V_CH0
- C45 pad 1: /Power Input & Regulation/+5V_CH3 -> /Power Input & Regulation/+5V_CH0
- C46 pad 1: /Power Input & Regulation/+5V_CH3 -> /Power Input & Regulation/+5V_CH0
- C63 pad 1: /Power Input & Regulation/+5V_CH2 -> /Power Input & Regulation/+5V_CH1
- C65 pad 1: /Power Input & Regulation/+5V_CH2 -> /Power Input & Regulation/+5V_CH1
- C68 pad 1: /Power Input & Regulation/+5V_CH2 -> /Power Input & Regulation/+5V_CH1
- C69 pad 1: /Power Input & Regulation/+5V_CH2 -> /Power Input & Regulation/+5V_CH1
- C71 pad 1: /Power Input & Regulation/+5V_CH2 -> /Power Input & Regulation/+5V_CH1
- C72 pad 1: /Power Input & Regulation/+5V_CH2 -> /Power Input & Regulation/+5V_CH1
- C89 pad 1: /Power Input & Regulation/+5V_CH0 -> /Power Input & Regulation/+5V_CH3
- C91 pad 1: /Power Input & Regulation/+5V_CH0 -> /Power Input & Regulation/+5V_CH3
- C94 pad 1: /Power Input & Regulation/+5V_CH0 -> /Power Input & Regulation/+5V_CH3
- C95 pad 1: /Power Input & Regulation/+5V_CH0 -> /Power Input & Regulation/+5V_CH3
- C97 pad 1: /Power Input & Regulation/+5V_CH0 -> /Power Input & Regulation/+5V_CH3
- C98 pad 1: /Power Input & Regulation/+5V_CH0 -> /Power Input & Regulation/+5V_CH3
- J2 pad 7: Net-(J2-Pad7) -> GND
- L10 pad 1: /Power Input & Regulation/+5V_CH1 -> /Power Input & Regulation/+5V_CH2
- L3 pad 1: /Power Input & Regulation/+5V_CH3 -> /Power Input & Regulation/+5V_CH0
- L4 pad 1: /Power Input & Regulation/+5V_CH3 -> /Power Input & Regulation/+5V_CH0
- L5 pad 1: /Power Input & Regulation/+5V_CH2 -> /Power Input & Regulation/+5V_CH1
- L6 pad 1: /Power Input & Regulation/+5V_CH2 -> /Power Input & Regulation/+5V_CH1
- L7 pad 1: /Power Input & Regulation/+5V_CH0 -> /Power Input & Regulation/+5V_CH3
- L8 pad 1: /Power Input & Regulation/+5V_CH0 -> /Power Input & Regulation/+5V_CH3
- L9 pad 1: /Power Input & Regulation/+5V_CH1 -> /Power Input & Regulation/+5V_CH2
- RN1 pad 1: /RF_ch0/I2C_SCL_ATTN -> /RF_ch1/I2C_SCL_ATTN
- RN1 pad 2: /RF_ch0/I2C_SDA_ATTN -> /RF_ch1/I2C_SDA_ATTN
- RN1 pad 3: /RF_ch1/I2C_SCL_ATTN -> /RF_ch0/I2C_SCL_ATTN
- RN1 pad 4: /RF_ch1/I2C_SDA_ATTN -> /RF_ch0/I2C_SDA_ATTN
- RN2 pad 1: /RF_ch2/I2C_SCL_ATTN -> /RF_ch3/I2C_SCL_ATTN
- RN2 pad 2: /RF_ch2/I2C_SDA_ATTN -> /RF_ch3/I2C_SDA_ATTN
- RN2 pad 3: /RF_ch3/I2C_SCL_ATTN -> /RF_ch2/I2C_SCL_ATTN
- RN2 pad 4: /RF_ch3/I2C_SDA_ATTN -> /RF_ch2/I2C_SDA_ATTN
- RN3 pad 1: /Digitial I/O via PMOD/INA219_PWR_MON_SCL -> /Digitial I/O via PMOD/EEPROM_SCL
- RN3 pad 2: /Digitial I/O via PMOD/INA219_PWR_MON_SDA -> /Digitial I/O via PMOD/EEPROM_SDA
- RN3 pad 3: /Digitial I/O via PMOD/EEPROM_SCL -> /Digitial I/O via PMOD/INA219_PWR_MON_SCL
- RN3 pad 4: /Digitial I/O via PMOD/EEPROM_SDA -> /Digitial I/O via PMOD/INA219_PWR_MON_SDA
- U16 pad 1: Net-(C50-Pad2) -> Net-(C49-Pad2)
- U16 pad 3: Net-(C49-Pad2) -> Net-(C50-Pad2)
- U16 pad 4: /RF_ch0/~1ST_NYQ~_2ND_NYQ_SW_INV -> /RF_ch0/~1ST_NYQ~_2ND_NYQ_SW
- U16 pad 6: /RF_ch0/~1ST_NYQ~_2ND_NYQ_SW -> /RF_ch0/~1ST_NYQ~_2ND_NYQ_SW_INV
- U24 pad 1: Net-(C76-Pad2) -> Net-(C75-Pad2)
- U24 pad 3: Net-(C75-Pad2) -> Net-(C76-Pad2)
- U24 pad 4: /RF_ch0/~1ST_NYQ~_2ND_NYQ_SW_INV -> /RF_ch0/~1ST_NYQ~_2ND_NYQ_SW
- U24 pad 6: /RF_ch0/~1ST_NYQ~_2ND_NYQ_SW -> /RF_ch0/~1ST_NYQ~_2ND_NYQ_SW_INV
- U32 pad 1: Net-(C102-Pad2) -> Net-(C101-Pad2)
- U32 pad 3: Net-(C101-Pad2) -> Net-(C102-Pad2)
- U32 pad 4: /RF_ch0/~1ST_NYQ~_2ND_NYQ_SW_INV -> /RF_ch0/~1ST_NYQ~_2ND_NYQ_SW
- U32 pad 6: /RF_ch0/~1ST_NYQ~_2ND_NYQ_SW -> /RF_ch0/~1ST_NYQ~_2ND_NYQ_SW_INV
- U40 pad 1: Net-(C128-Pad2) -> Net-(C127-Pad2)
- U40 pad 3: Net-(C127-Pad2) -> Net-(C128-Pad2)
- U40 pad 4: /RF_ch0/~1ST_NYQ~_2ND_NYQ_SW_INV -> /RF_ch0/~1ST_NYQ~_2ND_NYQ_SW
- U40 pad 6: /RF_ch0/~1ST_NYQ~_2ND_NYQ_SW -> /RF_ch0/~1ST_NYQ~_2ND_NYQ_SW_INV
- U7 pad 17: Net-(U7-Pad17) -> GND
- U7 pad 18: Net-(U7-Pad18) -> GND
- U7 pad 19: Net-(U7-Pad19) -> GND
- U7 pad 20: Net-(U7-Pad20) -> GND
Routing:
- net +3V3: track 13.0 -> 99.3 mm, vias 5 -> 24
- net /Digitial I/O via PMOD/INA219_PWR_MON_SDA: track 0.00 -> 51.9 mm, vias 0 -> 1
- net /Digitial I/O via PMOD/INA219_PWR_MON_SCL: track 0.00 -> 50.0 mm, vias 0 -> 1
- net GND: track 24.8 -> 74.4 mm, vias 27 -> 1191
- net /RF_ch3/LE_TX: track 0.00 -> 32.2 mm, vias 0 -> 1
- net /RF_ch2/LE_TX: track 0.00 -> 32.2 mm, vias 0 -> 1
- net /RF_ch0/LE_TX: track 0.00 -> 32.2 mm, vias 0 -> 1
- net /RF_ch1/LE_TX: track 0.00 -> 32.2 mm, vias 0 -> 1
- net /RF_ch3/LE_RX: track 0.00 -> 27.6 mm, vias 0 -> 1
- net /RF_ch1/LE_RX: track 0.00 -> 27.6 mm, vias 0 -> 1
- net /RF_ch0/LE_RX: track 0.00 -> 27.6 mm, vias 0 -> 1
- net /RF_ch2/LE_RX: track 0.00 -> 27.6 mm, vias 0 -> 1
- net /RF_ch3/C16_RX: track 0.00 -> 21.0 mm, vias 0 -> 1
- net /RF_ch1/C16_RX: track 0.00 -> 21.0 mm, vias 0 -> 1
- net /RF_ch0/C16_RX: track 0.00 -> 21.0 mm, vias 0 -> 1
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- added copper zone on F.Cu, net +3V3
- added copper zone on F.Cu, net /Power Input & Regulation/+5V_CH0
- added copper zone on F.Cu, net /Power Input & Regulation/+5V_CH1
- added copper zone on B.Cu, net /Power Input & Regulation/+5V_CH2
- added copper zone on F.Cu, net /Power Input & Regulation/+5V_CH2
- added copper zone on B.Cu, net /Power Input & Regulation/+5V_CH3
- added copper zone on F.Cu, net /Power Input & Regulation/+5V_CH3
- added copper zone on B.Cu, net /Power Input & Regulation/5V5_SW
- added copper zone on B.Cu, net GND

Commit message: more optimized RF layout, smaller overal layout
Signed-off-by: Gentile, John <johncgentile17@gmail.com>
Parts:
- moved J16 121.9 mm to (273.0, 186.9)
- moved C109 121.9 mm to (270.4, 179.3)
- moved H3 121.8 mm to (284.5, 102.4)
- moved H4 121.2 mm to (284.5, 186.9)
- moved U27 118.0 mm to (267.4, 121.1)
- moved C100 117.9 mm to (265.5, 138.5)
- moved C101 117.9 mm to (264.9, 150.8)
- moved C102 117.9 mm to (269.5, 149.5)
- moved C105 117.9 mm to (264.9, 157.4)
- moved C108 117.9 mm to (267.3, 166.2)
- moved C92 117.9 mm to (263.6, 128.0)
- moved C96 117.9 mm to (265.7, 127.7)
- moved F12 117.9 mm to (265.3, 154.5)
- moved U31 117.9 mm to (264.3, 133.0)
- moved U32 117.9 mm to (267.2, 144.1)
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Routing:
- net /RF_ch2/LE_TX: track 32.2 -> 16.8 mm, vias 1 -> 3
- net /RF_ch0/LE_TX: track 32.2 -> 16.8 mm, vias 1 -> 3
- net /RF_ch3/LE_TX: track 32.2 -> 16.8 mm, vias 1 -> 3
- net /RF_ch1/LE_TX: track 32.2 -> 16.8 mm, vias 1 -> 3
- net /RF_ch3/C1_RX: track 20.8 -> 15.1 mm
- net /RF_ch2/C1_RX: track 20.8 -> 15.1 mm
- net /RF_ch0/C1_RX: track 20.8 -> 15.1 mm
- net /RF_ch1/C1_RX: track 20.8 -> 15.1 mm
- net /RF_ch3/C2_RX: track 20.9 -> 15.1 mm
- net /RF_ch0/C2_RX: track 20.9 -> 15.1 mm
- net /RF_ch3/C1_TX: track 18.9 -> 13.1 mm
- net /RF_ch2/C2_RX: track 20.9 -> 15.1 mm
- net /RF_ch3/C4_TX: track 18.7 -> 13.0 mm
- net /RF_ch3/C16_TX: track 18.6 -> 12.9 mm
- net /RF_ch3/C2_TX: track 18.8 -> 13.1 mm
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
Commit message: final layout
Signed-off-by: Gentile, John <johncgentile17@gmail.com>
Parts:
- added DS2: LTST-C190KGKT, digikey-footprints:LED_0603, F.Cu at (58.7, 182.1)
- added R31: 75, Resistor_SMD:R_0603_1608Metric_Pad1.05x0.95mm_HandSolder, F.Cu at (58.7, 186.6)
- L2: value SRR6038-3R3Y -> IND_BOURNS_SRR6038
- U1, U2, U3, U4: value MCP1755ST-5002E_DB -> SOT-223_3MC
- U10: value SN74HCU04PWR -> PW14
- U11, U14, U19, U22, U27, U30, U35, U38: value ADL5611ARKZ-R7 -> RK_3
- U6: value TPS562208DDCT -> DDC0006A_N
- U9: value SN74LVC125APWR -> PW14
- moved C10 6.35 mm to (64.5, 125.3)
- moved C16 6.35 mm to (64.5, 114.4)
- moved C20 6.35 mm to (64.5, 111.4)
- moved C24 6.35 mm to (64.5, 108.2)
- moved C28 6.35 mm to (64.1, 184.8)
- moved C31 6.35 mm to (71.1, 178.7)
- moved R16 6.35 mm to (67.2, 174.5)
- moved R18 6.35 mm to (67.2, 173.2)
- moved RN2 6.35 mm to (76.2, 176.1)
- moved C1 6.35 mm to (52.1, 143.4)
- moved C11 6.35 mm to (63.1, 151.1)
- moved C12 6.35 mm to (60.5, 140.8)
- moved C13 6.35 mm to (56.0, 114.4)
- moved C14 6.35 mm to (66.5, 108.2)
- moved C15 6.35 mm to (51.1, 108.2)
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Connections:
- RN1 pad 1: /RF_ch1/I2C_SCL_ATTN -> /RF_ch2/I2C_SCL_ATTN
- RN1 pad 2: /RF_ch1/I2C_SDA_ATTN -> /RF_ch2/I2C_SDA_ATTN
- RN1 pad 3: /RF_ch0/I2C_SCL_ATTN -> /RF_ch3/I2C_SCL_ATTN
- RN1 pad 4: /RF_ch0/I2C_SDA_ATTN -> /RF_ch3/I2C_SDA_ATTN
- RN2 pad 1: /RF_ch3/I2C_SCL_ATTN -> /RF_ch0/I2C_SCL_ATTN
- RN2 pad 2: /RF_ch3/I2C_SDA_ATTN -> /RF_ch0/I2C_SDA_ATTN
- RN2 pad 3: /RF_ch2/I2C_SCL_ATTN -> /RF_ch1/I2C_SCL_ATTN
- RN2 pad 4: /RF_ch2/I2C_SDA_ATTN -> /RF_ch1/I2C_SDA_ATTN
- U7 pad 10: /RF_ch3/I2C_SDA_ATTN -> /RF_ch0/I2C_SDA_ATTN
- U7 pad 11: /RF_ch3/I2C_SCL_ATTN -> /RF_ch0/I2C_SCL_ATTN
- U7 pad 4: /RF_ch0/I2C_SDA_ATTN -> /RF_ch3/I2C_SDA_ATTN
- U7 pad 5: /RF_ch0/I2C_SCL_ATTN -> /RF_ch3/I2C_SCL_ATTN
- U7 pad 6: /RF_ch1/I2C_SDA_ATTN -> /RF_ch2/I2C_SDA_ATTN
- U7 pad 7: /RF_ch1/I2C_SCL_ATTN -> /RF_ch2/I2C_SCL_ATTN
- U7 pad 8: /RF_ch2/I2C_SDA_ATTN -> /RF_ch1/I2C_SDA_ATTN
- U7 pad 9: /RF_ch2/I2C_SCL_ATTN -> /RF_ch1/I2C_SCL_ATTN
Routing:
- net /RF_ch0/~1ST_NYQ~_2ND_NYQ_SW: track 0.00 -> 336.0 mm, vias 0 -> 9
- net /RF_ch0/~1ST_NYQ~_2ND_NYQ_SW_INV: track 0.00 -> 326.0 mm, vias 0 -> 9
- net /Digitial I/O via PMOD/~RX~_TX_SW3_INV: track 1.42 -> 238.8 mm, vias 1 -> 3
- net /RF_ch3/~RX~_TX_SW: track 0.00 -> 230.4 mm, vias 0 -> 2
- net /RF_ch3/I2C_SDA_ATTN: track 4.04 -> 227.3 mm
- net /RF_ch3/I2C_SCL_ATTN: track 3.27 -> 223.7 mm
- net /Digitial I/O via PMOD/~RX~_TX_SW2_INV: track 0.00 -> 191.1 mm, vias 0 -> 2
- net /RF_ch2/~RX~_TX_SW: track 0.00 -> 179.4 mm, vias 0 -> 2
- net /RF_ch2/I2C_SDA_ATTN: track 5.57 -> 176.7 mm
- net /RF_ch2/I2C_SCL_ATTN: track 4.80 -> 173.1 mm
- net /Digitial I/O via PMOD/~RX~_TX_SW1_INV: track 0.00 -> 141.2 mm, vias 0 -> 4
- net /RF_ch1/~RX~_TX_SW: track 0.00 -> 134.3 mm, vias 0 -> 2
- net /RF_ch1/I2C_SCL_ATTN: track 6.68 -> 119.2 mm
- net /RF_ch1/I2C_SDA_ATTN: track 7.45 -> 116.2 mm
- net /Digitial I/O via PMOD/~RX~_TX_SW0_INV: track 0.00 -> 88.5 mm, vias 0 -> 4
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- added copper zone on PWR.Cu, net +3V3
- added copper zone on PWR.Cu, net /Power Input & Regulation/+5V_CH0
- added copper zone on PWR.Cu, net /Power Input & Regulation/+5V_CH1
- added copper zone on PWR.Cu, net /Power Input & Regulation/+5V_CH2
- added copper zone on PWR.Cu, net /Power Input & Regulation/+5V_CH3
- added copper zone on GND.Cu, net GND
Other:
- board outline added: 249.9 x 94.7 mm

Commit message: (+) final silkscreen changes
Signed-off-by: Gentile, John <johncgentile17@gmail.com>
Parts:
- added G***: LOGO, jcg_custom:JHU_logo_small_low_DPI, F.Cu at (74.6, 101.0)
- added REF**: OSHW-Symbol_6.7x6mm_SilkScreen, Symbol:OSHW-Symbol_6.7x6mm_SilkScreen, F.Cu at (67.3, 101.0)
- added REF**: ESD-Logo_6.6x6mm_SilkScreen, Symbol:ESD-Logo_6.6x6mm_SilkScreen, F.Cu at (59.8, 101.2)
- added REF**: Symbol_Barrel_Polarity, Symbol:Symbol_Barrel_Polarity, F.Cu at (44.2, 157.2)
- moved FID1 5.60 mm to (279.6, 178.7)
- moved FID2 5.60 mm to (283.4, 178.7)
- moved FID3 5.60 mm to (283.4, 174.9)
Other:
- board text added: "+"
- board text added: "+9-12V"
- board text added: "-"
- board text added: "4-Channel RF Front End JCG-0 Rev. A"
- board text added: "ANT 0"
- board text added: "ANT 1"
- board text added: "ANT 2"
- board text added: "ANT 3"
- board text added: "RX 0(+)"
- board text added: "RX 0(-)"
- board text added: "RX 1(+)"
- board text added: "RX 1(-)"
- board text added: "RX 2(+)"
- board text added: "RX 2(-)"
- board text added: "RX 3(+)"
- board text added: "RX 3(-)"
- board text added: "TX 0(+)"
- board text added: "TX 0(-)"
- board text added: "TX 1(+)"
- board text added: "TX 1(-)"
- board text added: "TX 2(+)"
- board text added: "TX 2(-)"
- board text added: "TX 3(+)"
- board text added: "TX 3(-)"
